File: hardware/base_prototype/pcb/ledboard.sch (KiCad schematic (older format))
At the start: 57 parts, among them CON1 BARREL_JACK, P1 CONN_2, P2 CONN_2, P3 CONN_01X05, P4 PIR SENSOR, P5 CONN_01X03, P6 CONN_2, P7 CONN_2, P8 CONN_2, Q1 IRF540N, Q2 IRF540N, Q3 IRF540N, SW1 SW_PUSH, U1 LM1117-3.3, U2 ESP-12E, U3 FAN3100TSX, U4 FAN3100TSX, U5 FAN3100TSX, U6 NC R-78E3.3-0.5

Commit message: Converted RAY into suntracker
Parts:
- C1, C16: symbol CAPAPOL -> ledboard-rescue:CAPAPOL
- C10, C11, C12, C13, C14, C15, C2, C6, C7, C8, C9: symbol C_Small -> Device:C_Small
- CON1: symbol BARREL_JACK -> ledboard-rescue:BARREL_JACK
- D4: symbol LED -> ledboard-rescue:LED
- D?: symbol D -> Device:D
- P1, P2, P6, P7, P8: symbol CONN_2 -> ledboard-rescue:CONN_2
- P3: symbol CONN_01X05 -> ledboard-rescue:CONN_01X05
- P4, P5: symbol CONN_01X03 -> ledboard-rescue:CONN_01X03
- Q1, Q2, Q3: symbol IRF540N -> ledboard-rescue:IRF540N
- R1, R10, R11, R12, R13, R14, R15, R16, R17, R18, R2, R4, R5, R6, R7, R8, R9, R? (x2): symbol R -> Device:R
- SW1: symbol SW_PUSH -> ledboard-rescue:SW_PUSH
- U1: symbol LM1117-3.3 -> ledboard-rescue:LM1117-3.3
- U2: symbol ESP-12E -> ESP8266:ESP-12E
- U3, U4, U5: symbol FAN3100TSX -> ledboard-rescue:FAN3100TSX
- U6: symbol LM7805CT -> ledboard-rescue:LM7805CT
- Z1, Z2, Z3, Z4: symbol MHOLE -> components:MHOLE
Connections:
- wire segments 128 -> 147
